File: pcc_v0.2.kicad_pcb (KiCad board)
At the start: 2 copper layers, 170.3 x 151.7 mm, 69 parts, among them J2 Conn_01x04_Socket, J3 Conn_01x02_Socket, J4 Conn_02x14_Counter_Clockwise, J6 Conn_01x04_Socket, J7 Conn_01x04_Socket, J8 Conn_01x02_Socket, K3 PCN-112D3MHZ_000, K4 Relay_SPDT, U10 LM2904B, U2 4N35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

Commit message: Add files via upload
Connections:
- J6 pad 3: TS- -> TS+
- J6 pad 4: TS+ -> TS-
- R21 pad 1: TS- -> TS+
Routing:
- net TS-: track 162.3 -> 134.6 mm
- net TS+: track 134.6 -> 162.3 mm
- net Net-(U10A-+): track 18.6 -> 17.9 mm

Commit message: Add files via upload
Parts:
- added C14: 100n, Capacitor_SMD:C_0805_2012Metric, F.Cu at (108.2, 101.0)
- added C15: 100n, Capacitor_SMD:C_0805_2012Metric, F.Cu at (117.0, 102.2)
- added C16: 100n, Capacitor_SMD:C_0805_2012Metric, F.Cu at (113.0, 89.5)
- added C17: 100n, Capacitor_SMD:C_0805_2012Metric, F.Cu at (125.8, 93.8)
- added D3: RF01VM2S, Diode_SMD:D_SOD-323, F.Cu at (64.4, 96.9)
- added D4: ESD562-Q1, Package_TO_SOT_SMD:SOT-23-3, F.Cu at (73.5, 83.9)
- added F1: Fuse, Fuse:Fuse_1206_3216Metric, F.Cu at (205.5, 43.8)
- added F2: Fuse, Fuse:Fuse_1206_3216Metric, F.Cu at (201.9, 52.4)
- added J5: Conn_01x02_Socket, Connector_Molex:Molex_Mini-Fit_Jr_5566-02A2_2x01_P4.20mm_Vertical, F.Cu at (218.3, 52.8)
- added K5: PCN-112D3MHZ_000, PCN_112D3HMZ:RELAY_PCN-105D3MHZ_000_TEC, F.Cu at (70.8, 93.2)
- added Q1: MMBT3906, Package_TO_SOT_SMD:SOT-23, F.Cu at (91.1, 102.5)
- added Q2: MMBT3906, Package_TO_SOT_SMD:SOT-23, F.Cu at (90.3, 90.7)
- added R34: 500k, Resistor_SMD:R_0805_2012Metric, F.Cu at (113.8, 102.2)
- added R35: 10k, Resistor_SMD:R_0805_2012Metric, F.Cu at (121.2, 97.5)
- added R36: 12k, Resistor_SMD:R_0805_2012Metric, F.Cu at (108.2, 97.8)
- added R37: 10k, Resistor_SMD:R_0805_2012Metric, F.Cu at (120.2, 102.2)
- added R38: 10k, Resistor_SMD:R_0805_2012Metric, F.Cu at (91.2, 106.5)
- added R39: 10k, Resistor_SMD:R_0805_2012Metric, F.Cu at (93.0, 99.2)
- added R40: 6k8, Resistor_SMD:R_0805_2012Metric, F.Cu at (69.0, 58.0)
- added R41: 2k2, Resistor_SMD:R_0805_2012Metric, F.Cu at (108.5, 105.5)
- added R42: 20k, Resistor_SMD:R_0805_2012Metric, F.Cu at (69.0, 61.5)
- added R43: R, Resistor_THT:R_Axial_DIN0207_L6.3mm_D2.5mm_P7.62mm_Horizontal, F.Cu at (106.4, 110.8)
- added R44: 12k, Resistor_SMD:R_0805_2012Metric, F.Cu at (108.0, 88.5)
- added R45: 10k, Resistor_SMD:R_0805_2012Metric, F.Cu at (122.5, 93.8)
- added R46: R, Resistor_THT:R_Axial_DIN0207_L6.3mm_D2.5mm_P7.62mm_Horizontal, F.Cu at (111.4, 85.0)
- added R47: 10k, Resistor_SMD:R_0805_2012Metric, F.Cu at (116.8, 89.5)
- added R48: 500k, Resistor_SMD:R_0805_2012Metric, F.Cu at (119.0, 93.7)
- added R49: 2k2, Resistor_SMD:R_0805_2012Metric, F.Cu at (108.2, 93.0)
- added R50: 10k, Resistor_SMD:R_0805_2012Metric, F.Cu at (90.3, 94.7)
- added R51: 10k, Resistor_SMD:R_0805_2012Metric, F.Cu at (92.3, 88.5)
- added R52: 20k, Resistor_SMD:R_0805_2012Metric, F.Cu at (69.0, 54.3)
- added R53: 6k8, Resistor_SMD:R_0805_2012Metric, F.Cu at (69.0, 50.7)
- added R54: 5k, Resistor_SMD:R_2512_6332Metric, F.Cu at (178.3, 52.5)
- added R55: 20k, Resistor_SMD:R_0805_2012Metric, B.Cu at (70.1, 43.2)
- added R56: 6k8, Resistor_SMD:R_0805_2012Metric, B.Cu at (70.1, 47.0)
- added R57: 5k, Resistor_SMD:R_2512_6332Metric, F.Cu at (186.8, 52.5)
- added R58: 5k, Resistor_SMD:R_2512_6332Metric, F.Cu at (195.3, 52.5)
- added R59: 5k, Resistor_SMD:R_2512_6332Metric, F.Cu at (181.8, 43.8)
- added R60: 5k, Resistor_SMD:R_2512_6332Metric, F.Cu at (190.2, 43.8)
- added R61: 5k, Resistor_SMD:R_2512_6332Metric, F.Cu at (198.5, 43.8)
- added U11: LM393, Package_SO:SOIC-8_3.9x4.9mm_P1.27mm, F.Cu at (114.8, 95.5)
- added U12: 4N35, Package_DIP:DIP-6_W7.62mm_Socket, F.Cu at (104.2, 105.6)
- added U13: DMN63D8L-7, nmos:SOIC_63D8L-7_DIO, F.Cu at (69.5, 86.5)
- added U14: 4N35, Package_DIP:DIP-6_W7.62mm_Socket, F.Cu at (104.3, 92.5)
- added U15: DMN63D8L-7, nmos:SOIC_63D8L-7_DIO, F.Cu at (83.5, 145.6)
- moved D2 16.9 mm to (84.8, 94.5)
- moved K3 8.29 mm to (82.1, 93.2)
- moved U5 5.55 mm to (79.2, 88.0)
- moved C12 3.31 mm to (69.8, 79.4)
- moved R31 3.31 mm to (84.6, 81.8)
- moved C10 3.31 mm to (83.9, 78.9)
- moved R27 3.31 mm to (73.5, 80.4)
- moved R33 3.31 mm to (73.5, 78.4)
- moved R30 3.31 mm to (84.6, 76.1)
- moved U8 3.31 mm to (79.0, 79.3)
- moved R32 2.06 mm to (77.5, 83.8)
Connections:
- D1 pad 2: GLV- -> Net-(D1-A)
- J4 pad 12: unconnected-(J4-Pin_12-Pad12) -> Pre_Dis
- J4 pad 14: unconnected-(J4-Pin_14-Pad14) -> IR-
- J8 pad 1: GLV- -> IR-_GND
- K4 pad A2: GLV- -> Net-(D1-A)
Routing:
- net TS+: track 162.3 -> 265.2 mm
- net +12P: track 146.5 -> 245.4 mm, vias 1 -> 2
- net Pre_Dis: track 0.00 -> 90.1 mm, vias 0 -> 1
- net GNDS: track 226.8 -> 305.6 mm
- net PDOC_OK1: track 0.00 -> 59.3 mm, vias 0 -> 2
- net PDOC_OK2: track 0.00 -> 49.1 mm, vias 0 -> 2
- net +12V: track 101.6 -> 146.8 mm
- net IR-_GND: track 0.00 -> 36.1 mm
- net Net-(U11A--): track 0.00 -> 27.5 mm, vias 0 -> 1
- net TS-: track 134.6 -> 157.4 mm
- net Net-(U11B-+): track 0.00 -> 21.6 mm, vias 0 -> 2
- net TSMP-: track 0.00 -> 18.8 mm
- net Net-(U11A-+): track 0.00 -> 17.3 mm, vias 0 -> 2
- net Net-(D3-A): track 0.00 -> 17.3 mm
- net IR-: track 0.00 -> 16.1 mm, vias 0 -> 1
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
Commit message: Add files via upload
Routing:
- net CANH: track 53.3 -> 54.9 mm
- net CANL: track 48.7 -> 49.9 mm
Changed lines of the file:
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@@
 		(tags "SOIC SO")
 		(property "Reference" "U8"
-			(at 0 -3.4 0)
+			(at 0 3.5225 0)
 			(layer "F.SilkS")
 			(effects
@@
 		(tags "resistor")
 		(property "Reference" "R32"
-			(at 0.1175 1.75 90)
+			(at 0 -1.75 90)
 			(layer "F.SilkS")
 			(effects
@@
 	)
 	(segment
-		(start 73.6115 79.181)
-		(end 73.6115 81.6635)
+		(start 73.5 90.8756)
+		(end 73.5 97.876994)
 		(width 0.2)
 		(layer "F.Cu")
@@
 	)
 	(segment
-		(start 65.199747 111.050253)
-		(end 65.199747 106.177247)
+		(start 73.6115 79.181)
+		(end 73.6115 81.6635)
 		(width 0.2)
 		(layer "F.Cu")
@@
 	)
 	(segment
-		(start 72.85 98.526994)
-		(end 72.563497 98.813497)
+		(start 76.28 78.3675)
+		(end 76.55 78.6375)
 		(width 0.2)
 		(layer "F.Cu")
@@
 	)
 	(segment
-		(start 76.28 78.3675)
-		(end 76.55 78.6375)
+		(start 73.6115 81.6635)
+		(end 72.55 82.725)
 		(width 0.2)
 		(layer "F.Cu")
@@
 	)
 	(segment
-		(start 73.6115 81.6635)
-		(end 72.55 82.725)
+		(start 65.199747 111.050253)
+		(end 58.322753 117.927247)
 		(width 0.2)
 		(layer "F.Cu")
@@
 	)
 	(segment
-		(start 72.85 83.025)
-		(end 72.85 98.526994)
+		(start 71.75 83.525)
+		(end 71.75 89.1256)
 		(width 0.2)
 		(layer "F.Cu")
@@
 	)
 	(segment
-		(start 65.199747 106.177247)
-		(end 72.563497 98.813497)
+		(start 71.75 89.1256)
+		(end 73.5 90.8756)
 		(width 0.2)
 		(layer "F.Cu")
@@
 	)
 	(segment
-		(start 58.322753 117.927247)
-		(end 65.199747 111.050253)
+		(start 73.5 97.876994)
+		(end 65.199747 106.177247)
 		(width 0.2)
 		(layer "F.Cu")
@@
 	(segment
 		(start 72.55 82.725)
-		(end 72.85 83.025)
+		(end 71.75 83.525)
+		(width 0.2)
+		(layer "F.Cu")
+		(net 9)
+	)
+	(segment
+		(start 65.199747 106.177247)
+		(end 65.199747 111.050253)
 		(width 0.2)
 		(layer "F.Cu")
@@
 	)
 	(segment
+		(start 75.5 111)
+		(end 66.25 120.25)
+		(width 0.2)
+		(layer "F.Cu")
+		(net 10)
+	)
+	(segment
 		(start 74.425 80.3675)
 		(end 76.09 80.3675)
@@
 	)
 	(segment
-		(start 66.922753 119.577247)
-		(end 60.872753 119.577247)
+		(start 60.2 120.25)
+		(end 58.5 121.95)
 		(width 0.2)
 		(layer "F.Cu")
@@
 	)
 	(segment
-		(start 60.872753 119.577247)
-		(end 58.5 121.95)
+		(start 74.425 80.3675)
+		(end 74.425 82.7)
+		(width 0.2)
+		(layer "F.Cu")
+		(net 10)
+	)
+	(segment
+		(start 74.425 82.7)
+		(end 74.45 82.725)
+		(width 0.2)
+		(layer "F.Cu")
+		(net 10)
+	)
+	(segment
+		(start 75.5 83.775)
+		(end 75.5 111)
 		(width 0.2)
 		(layer "F.Cu")
@@
 	)
 	(segment
-		(start 74.425 112.075)
-		(end 74.425 81.0975)
+		(start 66.25 120.25)
+		(end 60.2 120.25)
 		(width 0.2)
 		(layer "F.Cu")
@@
 	)
 	(segment
-		(start 66.922753 119.577247)
-		(end 74.425 112.075)
+		(start 74.45 82.725)
+		(end 75.5 83.775)
 		(width 0.2)
 		(layer "F.Cu")
@@
 	)
 	(segment
-		(start 72.199747 94.383699)
-		(end 70.841099 95.742347)
+		(start 69.5 89)
+		(end 72.5 92)
 		(width 0.2)
 		(layer "F.Cu")
@@
 	)
 	(segment
-		(start 69.5 87.5)
-		(end 69.5573 87.5)
+		(start 72.5 94.083446)
+		(end 70.841099 95.742347)
 		(width 0.2)
 		(layer "F.Cu")
@@
 	)
 	(segment
-		(start 72.199747 90.142447)
-		(end 72.199747 94.383699)
+		(start 69.5 87.5)
+		(end 69.5 89)
 		(width 0.2)
 		(layer "F.Cu")
@@
 	)
 	(segment
-		(start 69.5573 87.5)
-		(end 72.199747 90.142447)
+		(start 72.5 92)
+		(end 72.5 94.083446)
 		(width 0.2)
 		(layer "F.Cu")

Commit message: Add files via upload
Parts:
- removed C16, C17: 100n, Capacitor_SMD:C_0805_2012Metric
- removed D2, D3: RF01VM2S, Diode_SMD:D_SOD-323
- removed F1: Fuse, Fuse:Fuse_1206_3216Metric
- removed J5: Conn_01x02_Socket, Connector_Molex:Molex_Mini-Fit_Jr_5566-02A2_2x01_P4.20mm_Vertical
- removed K3, K5: PCN-112D3MHZ_000, PCN_112D3HMZ:RELAY_PCN-105D3MHZ_000_TEC
- removed R34, R48: 500k, Resistor_SMD:R_0805_2012Metric
- removed R35, R37, R38, R39, R45, R47, R50, R51: 10k, Resistor_SMD:R_0805_2012Metric
- removed R36: 12k, Resistor_SMD:R_0805_2012Metric
- removed R41, R49: 2k2, Resistor_SMD:R_0805_2012Metric
- removed R42, R52: 20k, Resistor_SMD:R_0805_2012Metric
- removed R46: R, Resistor_THT:R_Axial_DIN0207_L6.3mm_D2.5mm_P7.62mm_Horizontal
- removed R54, R57, R58, R59, R60, R61: 5k, Resistor_SMD:R_2512_6332Metric
- removed U11: LM393, Package_SO:SOIC-8_3.9x4.9mm_P1.27mm
- removed U12, U14: 4N35, Package_DIP:DIP-6_W7.62mm_Socket
- removed U13, U5: DMN63D8L-7, nmos:SOIC_63D8L-7_DIO
- added D5: RF01VM2S, Diode_SMD:D_SOD-323, F.Cu at (64.5, 142.3)
- added D6: RF01VM2S, Diode_SMD:D_SOD-323, F.Cu at (64.5, 145.2)
- added F3: Fuse, Fuse:Fuse_1206_3216Metric, F.Cu at (195.8, 39.8)
- added J9: Conn_01x04_Socket, Connector_Molex:Molex_Mini-Fit_Jr_5566-04A2_2x02_P4.20mm_Vertical, F.Cu at (218.8, 42.5)
- added R62: 3k, Resistor_SMD:R_2512_6332Metric, F.Cu at (168.2, 56.0)
- added R63: 3k, Resistor_SMD:R_2512_6332Metric, F.Cu at (172.8, 45.8)
- added R64: 3k, Resistor_SMD:R_2512_6332Metric, F.Cu at (176.0, 56.0)
- added R65: 3k, Resistor_SMD:R_2512_6332Metric, F.Cu at (180.5, 45.8)
- added R66: 4k, Resistor_SMD:R_0805_2012Metric, F.Cu at (210.0, 56.5)
- added R67: 4k, Resistor_SMD:R_0805_2012Metric, F.Cu at (191.1, 39.8)
- added R68: 3k, Resistor_SMD:R_2512_6332Metric, F.Cu at (183.8, 56.0)
- added R69: 3k, Resistor_SMD:R_2512_6332Metric, F.Cu at (188.3, 45.8)
- added R70: 3k, Resistor_SMD:R_2512_6332Metric, F.Cu at (191.5, 56.0)
- added R71: 3k, Resistor_SMD:R_2512_6332Metric, F.Cu at (196.0, 45.8)
- added R72: 3k, Resistor_SMD:R_2512_6332Metric, F.Cu at (199.5, 56.0)
- added R73: 3k, Resistor_SMD:R_2512_6332Metric, F.Cu at (203.8, 45.8)
- Q1, Q2: value MMBT3906 -> IRLZ44N; footprint Package_TO_SOT_SMD:SOT-23 -> Package_TO_SOT_THT:TO-220-3_Vertical
- R43: footprint Resistor_THT:R_Axial_DIN0207_L6.3mm_D2.5mm_P7.62mm_Horizontal -> Connector_PinSocket_2.00mm:PinSocket_1x02_P2.00mm_Vertical
- R44: value 12k -> R; footprint Resistor_SMD:R_0805_2012Metric -> Connector_PinSocket_2.00mm:PinSocket_1x02_P2.00mm_Vertical
- moved C15 73.0 mm to (65.2, 50.8), turned to 90 degrees
- moved C14 58.3 mm to (64.8, 62.2), turned to 90 degrees
- moved R43 57.2 mm to (68.5, 68.0), turned to 180 degrees
- moved R44 50.4 mm to (69.0, 56.5), turned to 180 degrees
- moved Q1 26.8 mm to (66.5, 91.8), turned to -90 degrees
- moved F2 13.2 mm to (214.5, 56.5)
- moved Q2 10.8 mm to (79.6, 91.0), turned to -90 degrees
- moved R40 4.37 mm to (68.5, 62.3)
- moved U15 0.26 mm to (83.7, 145.7)
Connections:
- C14 pad 1: +12P -> Net-(C14-Pad1)
- C14 pad 2: Net-(U11A--) -> GLV-
- C15 pad 1: Net-(U11A-+) -> Net-(C15-Pad1)
- C15 pad 2: GNDS -> GLV-
- F2 pad 2: TSMP+ -> TSMP+_Fused
- J4 pad 12: Pre_Dis -> unconnected-(J4-Pin_12-Pad12)
- J4 pad 14: IR- -> PreDis_IR-
- Q1 pad 1: Net-(Q1-B) -> PreDis_IR-
- Q1 pad 2: PDOC_OK1 -> IR-_GND
- Q1 pad 3: +12V -> GLV-
- Q2 pad 1: Net-(Q2-B) -> IR+
- Q2 pad 2: PDOC_OK2 -> IR+_GND
- Q2 pad 3: +12V -> GLV-
- R40 pad 1: Net-(R40-Pad1) -> Net-(C14-Pad1)
- R43 pad 1: +12P -> +3.3V
- R43 pad 2: Net-(U11A--) -> Net-(C14-Pad1)
- R44 pad 1: +12P -> +3.3V
- R44 pad 2: Net-(U11B-+) -> Net-(C15-Pad1)
- R53 pad 1: Net-(R52-Pad2) -> Net-(C15-Pad1)
- U15 pad 1: Pre_Dis -> PreDis_IR-
Routing:
- net PreDis_IR-: track 0.00 -> 108.8 mm, vias 0 -> 1
- net +12V: track 146.8 -> 41.3 mm
- net +12P: track 245.4 -> 146.5 mm, vias 2 -> 1
- net Pre_Dis: track 90.1 -> 0.00 mm, vias 1 -> 0
- net GNDS: track 305.6 -> 227.6 mm
- net PDOC_OK1: track 59.3 -> 0.00 mm, vias 2 -> 0
- net TS+: track 265.2 -> 320.2 mm
- net PDOC_OK2: track 49.1 -> 0.00 mm, vias 2 -> 0
- net +3.3V: track 56.6 -> 102.7 mm
- net TSMP-_Fused: track 0.00 -> 30.0 mm
- net Net-(U11A--): track 27.5 -> 0.00 mm, vias 1 -> 0
- net TS-: track 157.4 -> 180.5 mm
- net Net-(U11B-+): track 21.6 -> 0.00 mm, vias 2 -> 0
- net IR+_GND: track 56.9 -> 77.2 mm
- net Net-(D3-A): track 17.5 -> 0.00 mm
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